File: kicad_docs/seven_segment_display.sch (KiCad schematic (older format))
At the start: 21 parts, among them Q1 MMBT3904, Q2 MMBT3904, Q3 MMBT3904, Q4 MMBT3904, U1 HDSP-7503, U11 74HC595, U2 HDSP-7503, U3 HDSP-7503, U4 HDSP-7503

Commit message: add EEPROM, big pcb re-design
Parts:
- Q1, Q2, Q3, Q4: footprint Package_TO_SOT_SMD:SOT-23_Handsoldering -> Package_TO_SOT_SMD:SOT-23
- R25: renamed from R37; value 1k -> 3k3; footprint Resistor_SMD:R_0805_2012Metric_Pad1.15x1.40mm_HandSolder -> Resistor_SMD:R_0603_1608Metric
- R26: renamed from R57; value R -> 330; footprint Resistor_SMD:R_0805_2012Metric_Pad1.15x1.40mm_HandSolder -> Resistor_SMD:R_0603_1608Metric
- R27: renamed from R58; value R -> 330; footprint Resistor_SMD:R_0805_2012Metric_Pad1.15x1.40mm_HandSolder -> Resistor_SMD:R_0603_1608Metric
- R28: renamed from R59; value R -> 330; footprint Resistor_SMD:R_0805_2012Metric_Pad1.15x1.40mm_HandSolder -> Resistor_SMD:R_0603_1608Metric
- R29: renamed from R60; value R -> 330; footprint Resistor_SMD:R_0805_2012Metric_Pad1.15x1.40mm_HandSolder -> Resistor_SMD:R_0603_1608Metric
- R30: renamed from R61; value R -> 330; footprint Resistor_SMD:R_0805_2012Metric_Pad1.15x1.40mm_HandSolder -> Resistor_SMD:R_0603_1608Metric
- R31: renamed from R62; value R -> 330; footprint Resistor_SMD:R_0805_2012Metric_Pad1.15x1.40mm_HandSolder -> Resistor_SMD:R_0603_1608Metric
- R32: renamed from R63; value R -> 330; footprint Resistor_SMD:R_0805_2012Metric_Pad1.15x1.40mm_HandSolder -> Resistor_SMD:R_0603_1608Metric
- R33: renamed from R64; value R -> 330; footprint Resistor_SMD:R_0805_2012Metric_Pad1.15x1.40mm_HandSolder -> Resistor_SMD:R_0603_1608Metric
- R34: renamed from R38; value 1k -> 3k3; footprint Resistor_SMD:R_0805_2012Metric_Pad1.15x1.40mm_HandSolder -> Resistor_SMD:R_0603_1608Metric
- R35: renamed from R39; value 1k -> 3k3; footprint Resistor_SMD:R_0805_2012Metric_Pad1.15x1.40mm_HandSolder -> Resistor_SMD:R_0603_1608Metric
- R36: renamed from R40; value 1k -> 3k3; footprint Resistor_SMD:R_0805_2012Metric_Pad1.15x1.40mm_HandSolder -> Resistor_SMD:R_0603_1608Metric
- renumbered U11 to U2, U2 to U3, U3 to U4, U4 to U5
Connections:
- net segment_A: now also R26.1; no longer R33.1
- net segment_B: now also R27.1; no longer R32.1
- net segment_C: now also R29.1; no longer R30.1
- net segment_D: now also R33.1; no longer R26.1
- net segment_DP: now also R31.1; no longer R28.1
- net segment_E: now also R32.1; no longer R27.1
- net segment_F: now also R28.1; no longer R31.1
- net segment_G: now also R30.1; no longer R29.1
- net seven_segment_clk_in renamed spi_clk_in
- net seven_segment_data_in renamed spi_data_in
- net seven_segment_en_in renamed spi_seven_segment_cs
