File: kicad_docs/spi_dacs_and_level_shifters.sch (KiCad schematic (older format))
At the start: 28 parts, among them U10 MCP4822, U7 TL072, U8 TL072, U9 MCP4822

Commit message: add EEPROM, big pcb re-design
Parts:
- C37: renamed from C22; value C -> 2n2
- C38: renamed from C21; value C -> 2n2
- C39: renamed from C23; value C -> 2n2
- C40: renamed from C24; value C -> 2n2
- C41: renamed from C26; value C -> 2n2
- C42: renamed from C25; value C -> 2n2
- C43: renamed from C27; value C -> 2n2
- C44: renamed from C28; value C -> 2n2
- R65: renamed from R66; value R -> 50k; footprint Resistor_SMD:R_0805_2012Metric_Pad1.15x1.40mm_HandSolder -> Resistor_SMD:R_0603_1608Metric
- R66: renamed from R65; value R -> 50k; footprint Resistor_SMD:R_0805_2012Metric_Pad1.15x1.40mm_HandSolder -> Resistor_SMD:R_0603_1608Metric
- R67: renamed from R68; value R -> 200k; footprint Resistor_SMD:R_0805_2012Metric_Pad1.15x1.40mm_HandSolder -> Resistor_SMD:R_0603_1608Metric
- R68: renamed from R67; value R -> 200k; footprint Resistor_SMD:R_0805_2012Metric_Pad1.15x1.40mm_HandSolder -> Resistor_SMD:R_0603_1608Metric
- R69, R70, R77, R78: value R -> 33k; footprint Resistor_SMD:R_0805_2012Metric_Pad1.15x1.40mm_HandSolder -> Resistor_SMD:R_0603_1608Metric
- R71, R72, R79, R80: value R -> 68k; footprint Resistor_SMD:R_0805_2012Metric_Pad1.15x1.40mm_HandSolder -> Resistor_SMD:R_0603_1608Metric
- R73: renamed from R74; value R -> 50k; footprint Resistor_SMD:R_0805_2012Metric_Pad1.15x1.40mm_HandSolder -> Resistor_SMD:R_0603_1608Metric
- R74: renamed from R73; value R -> 50k; footprint Resistor_SMD:R_0805_2012Metric_Pad1.15x1.40mm_HandSolder -> Resistor_SMD:R_0603_1608Metric
- R75: renamed from R76; value R -> 200k; footprint Resistor_SMD:R_0805_2012Metric_Pad1.15x1.40mm_HandSolder -> Resistor_SMD:R_0603_1608Metric
- R76: renamed from R75; value R -> 200k; footprint Resistor_SMD:R_0805_2012Metric_Pad1.15x1.40mm_HandSolder -> Resistor_SMD:R_0603_1608Metric
- renumbered U8 to U11, U7 to U8
Connections:
- net adsr_1_3.3v: now also U9.6 (VB); no longer U9.8 (VA)
- net adsr_2_3.3v: now also U9.8 (VA); no longer U9.6 (VB)
- net adsr_3_3.3v: now also U10.6 (VB); no longer U10.8 (VA)
- net adsr_4_3.3v: now also U10.8 (VA); no longer U10.6 (VB)
- net spi_cs_1_in renamed spi_dac1_cs
- net spi_cs_2_in renamed spi_dac2_cs
