File: hardware/main_pcb/kicad_docs/quad_adsr.kicad_pcb (KiCad board)
At the start: 4 copper layers, 71.1 x 99.1 mm, 197 parts, among them J1 PJ301M-12, J10 gate_3_in, J11 trigger_3_in, J12 gate_4_in, J13 trigger_4_in, J14 SWD_header, J2 PJ301M-12, J3 PJ301M-12, J4 PJ301M-12, J5 power_in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

Commit message: add pin 1 locations to silk
Other:
- board text added: "+"
